Commit message: Fix wujihand_left mano anchors (mirror row/col bug) + base_joint v4
Root cause: generator fitted mirror row-wise (p@M+t) but applied column-wise
(M@p+t); the simplified-right->vendor-left fit M is an oblique reflection
(not ~diag(1,-1,1)), displacing all 21 finger anchors 7-28cm off the links
(skeleton ~98deg from mesh; invisible to keypoint metrics).

- anchors: exact mirror of right model (offsets 0.5-4.4cm, on-mesh <=3mm
  at MCPs; skeleton-vs-mesh 97.8->2.6deg)
- base_joint v4: mirror-conjugate candidate + one-shot data fold-in
  G'=T_r^-1 T_off G (right baseline 4.7-6.4deg from 2 right demos)
- smoke verification (cut_knife_L 200f, Mosek): base<->wrist 5.39+/-0.72deg,
  |dp| 2.2mm, keypoint err 1.08cm, mesh visually overlaps MANO skeleton
- supersedes v2/v3 calibrations (measured with broken anchors)
See REGRIND/docs/lefthand_anchor_fix_20260922.md

File: source/regrind/regrind/assets/mjcf/free_wuji_left_hand_full_simplified_v1.urdf (robot description, URDF)
Before this commit: robot wujihand-left, 48 links, 47 joints
Joints:
- joint base_joint: origin xyz=0.004128 0.014200 0.044564 rpy=-2.699035 1.409043 1.624471 -> xyz=-0.023954 0.002647 -0.004772 rpy=-1.473021 0.120299 -1.695369
- joint mano_0: origin xyz=-0.000034 0.000031 0.020009 rpy=0 0 0 -> xyz=-0.000003 -0.000006 -0.000028 rpy=0 0 0
- joint mano_1: origin xyz=-0.005572 0.099079 -0.087173 rpy=0 0 0 -> xyz=0.002208 -0.000047 0.003982 rpy=0 0 0
- joint mano_10: origin xyz=0.013125 0.062086 -0.066257 rpy=0 0 0 -> xyz=0.002194 -0.000038 0.004013 rpy=0 0 0
- joint mano_11: origin xyz=0.105667 -0.012695 -0.069964 rpy=0 0 0 -> xyz=-0.000078 0.000029 0.043631 rpy=0 0 0
- joint mano_12: origin xyz=0.018531 0.135178 -0.118087 rpy=0 0 0 -> xyz=-0.000000 -0.000108 0.029514 rpy=0 0 0
- joint mano_13: origin xyz=-0.006845 0.018099 -0.053120 rpy=0 0 0 -> xyz=-0.004739 0.005784 0.014118 rpy=0 0 0
- joint mano_14: origin xyz=-0.041563 -0.067940 -0.059992 rpy=0 0 0 -> xyz=-0.000126 -0.000975 0.034635 rpy=0 0 0
- joint mano_15: origin xyz=-0.066908 0.089000 -0.101471 rpy=0 0 0 -> xyz=0.000018 0.000228 0.029469 rpy=0 0 0
- joint mano_16: origin xyz=-0.085992 0.110473 -0.140101 rpy=0 0 0 -> xyz=0.000014 0.000146 0.029968 rpy=0 0 0
- joint mano_17: origin xyz=0.004199 0.191145 -0.184031 rpy=0 0 0 -> xyz=0.000004 0.000063 0.020982 rpy=0 0 0
- joint mano_18: origin xyz=-0.002435 0.174741 -0.168241 rpy=0 0 0 -> xyz=0.000013 0.000068 0.020997 rpy=0 0 0
- joint mano_19: origin xyz=0.019389 0.156360 -0.147433 rpy=0 0 0 -> xyz=0.000001 0.000072 0.021014 rpy=0 0 0
- joint mano_2: origin xyz=0.141938 0.003802 -0.098237 rpy=0 0 0 -> xyz=-0.000087 -0.000006 0.043600 rpy=0 0 0
- joint mano_20: origin xyz=0.034198 0.135841 -0.120208 rpy=0 0 0 -> xyz=-0.000005 0.000077 0.022530 rpy=0 0 0
- joint mano_3: origin xyz=0.002282 0.170311 -0.151130 rpy=0 0 0 -> xyz=0.000005 -0.000117 0.029482 rpy=0 0 0
- joint mano_4: origin xyz=-0.003868 0.081203 -0.078176 rpy=0 0 0 -> xyz=0.002205 -0.000041 0.003997 rpy=0 0 0
- joint mano_5: origin xyz=0.124653 0.006420 -0.085992 rpy=0 0 0 -> xyz=-0.000082 -0.000009 0.043615 rpy=0 0 0
- joint mano_6: origin xyz=-0.002272 0.153622 -0.136904 rpy=0 0 0 -> xyz=0.000011 -0.000112 0.029497 rpy=0 0 0
- joint mano_7: origin xyz=0.027263 0.040311 -0.050616 rpy=0 0 0 -> xyz=0.002184 -0.000033 0.004029 rpy=0 0 0
- joint mano_8: origin xyz=0.083537 -0.026879 -0.049073 rpy=0 0 0 -> xyz=-0.000073 0.000044 0.043647 rpy=0 0 0
- joint mano_9: origin xyz=0.033256 0.113346 -0.093585 rpy=0 0 0 -> xyz=-0.000008 -0.000103 0.029530 rpy=0 0 0

File: source/regrind/regrind/assets/mjcf/free_wuji_left_hand_full_simplified_v1_render.urdf (robot description, URDF)
Before this commit: robot wujihand-left, 48 links, 47 joints
Joints:
- joint base_joint: origin xyz=0.004128 0.014200 0.044564 rpy=-2.699035 1.409043 1.624471 -> xyz=-0.023954 0.002647 -0.004772 rpy=-1.473021 0.120299 -1.695369
- joint mano_0: origin xyz=-0.000034 0.000031 0.020009 rpy=0 0 0 -> xyz=-0.000003 -0.000006 -0.000028 rpy=0 0 0
- joint mano_1: origin xyz=-0.005572 0.099079 -0.087173 rpy=0 0 0 -> xyz=0.002208 -0.000047 0.003982 rpy=0 0 0
- joint mano_10: origin xyz=0.013125 0.062086 -0.066257 rpy=0 0 0 -> xyz=0.002194 -0.000038 0.004013 rpy=0 0 0
- joint mano_11: origin xyz=0.105667 -0.012695 -0.069964 rpy=0 0 0 -> xyz=-0.000078 0.000029 0.043631 rpy=0 0 0
- joint mano_12: origin xyz=0.018531 0.135178 -0.118087 rpy=0 0 0 -> xyz=-0.000000 -0.000108 0.029514 rpy=0 0 0
- joint mano_13: origin xyz=-0.006845 0.018099 -0.053120 rpy=0 0 0 -> xyz=-0.004739 0.005784 0.014118 rpy=0 0 0
- joint mano_14: origin xyz=-0.041563 -0.067940 -0.059992 rpy=0 0 0 -> xyz=-0.000126 -0.000975 0.034635 rpy=0 0 0
- joint mano_15: origin xyz=-0.066908 0.089000 -0.101471 rpy=0 0 0 -> xyz=0.000018 0.000228 0.029469 rpy=0 0 0
- joint mano_16: origin xyz=-0.085992 0.110473 -0.140101 rpy=0 0 0 -> xyz=0.000014 0.000146 0.029968 rpy=0 0 0
- joint mano_17: origin xyz=0.004199 0.191145 -0.184031 rpy=0 0 0 -> xyz=0.000004 0.000063 0.020982 rpy=0 0 0
- joint mano_18: origin xyz=-0.002435 0.174741 -0.168241 rpy=0 0 0 -> xyz=0.000013 0.000068 0.020997 rpy=0 0 0
- joint mano_19: origin xyz=0.019389 0.156360 -0.147433 rpy=0 0 0 -> xyz=0.000001 0.000072 0.021014 rpy=0 0 0
- joint mano_2: origin xyz=0.141938 0.003802 -0.098237 rpy=0 0 0 -> xyz=-0.000087 -0.000006 0.043600 rpy=0 0 0
- joint mano_20: origin xyz=0.034198 0.135841 -0.120208 rpy=0 0 0 -> xyz=-0.000005 0.000077 0.022530 rpy=0 0 0
- joint mano_3: origin xyz=0.002282 0.170311 -0.151130 rpy=0 0 0 -> xyz=0.000005 -0.000117 0.029482 rpy=0 0 0
- joint mano_4: origin xyz=-0.003868 0.081203 -0.078176 rpy=0 0 0 -> xyz=0.002205 -0.000041 0.003997 rpy=0 0 0
- joint mano_5: origin xyz=0.124653 0.006420 -0.085992 rpy=0 0 0 -> xyz=-0.000082 -0.000009 0.043615 rpy=0 0 0
- joint mano_6: origin xyz=-0.002272 0.153622 -0.136904 rpy=0 0 0 -> xyz=0.000011 -0.000112 0.029497 rpy=0 0 0
- joint mano_7: origin xyz=0.027263 0.040311 -0.050616 rpy=0 0 0 -> xyz=0.002184 -0.000033 0.004029 rpy=0 0 0
- joint mano_8: origin xyz=0.083537 -0.026879 -0.049073 rpy=0 0 0 -> xyz=-0.000073 0.000044 0.043647 rpy=0 0 0
- joint mano_9: origin xyz=0.033256 0.113346 -0.093585 rpy=0 0 0 -> xyz=-0.000008 -0.000103 0.029530 rpy=0 0 0

Commit message: Regenerate left collision with right-hand budget (170->37 meshes)
Per-link coacd budgets mirror the official simplified right model
(palm=1, finger1_link1=2, finger{2-5}_link1=3, link2/3=1, link4=1,
pinky link4=2, tips=1). Smoke rerun metrics bit-identical (5.387deg,
1.0836cm); per-frame QP 1.35s -> 0.13s.

File: source/regrind/regrind/assets/mjcf/free_wuji_left_hand_full_simplified_v1.urdf (robot description, URDF)
Before this commit: robot wujihand-left, 48 links, 47 joints
Links:
- link left_finger1_link1: geometry collision mesh filename=./assets/wujihand_full_simplified_v1/left/left_finger1_link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; collision mesh filename=./assets/wujihand_full_simplified_v1/left/left_finger1_link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
- link left_finger1_link2: geometry collision mesh filename=./assets/wujihand_full_simplified_v1/left/left_finger1_link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; visual mesh filename=./assets/wujihand_full/left/left_finger1_link2.STL
- link left_finger1_link3: geometry collision mesh filename=./assets/wujihand_full_simplified_v1/left/left_finger1_link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; visual mesh filename=./assets/wujihand_full/left/left_finger1_link3.STL
- link left_finger1_link4: geometry collision mesh filename=./assets/wujihand_full_simplified_v1/left/left_finger1_link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; visual mesh filename=./assets/wujihand_full/left/left_finger1_link4.STL
- link left_finger2_link1: geometry collision mesh filename=./assets/wujihand_full_simplified_v1/left/left_finger2_link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; collision mesh filename=./assets/wujihand_full_simplified_v1/left/left_finger2_link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
- link left_finger2_link2: geometry collision mesh filename=./assets/wujihand_full_simplified_v1/left/left_finger2_link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; visual mesh filename=./assets/wujihand_full/left/left_finger2_link2.STL
- link left_finger2_link3: geometry collision mesh filename=./assets/wujihand_full_simplified_v1/left/left_finger2_link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; visual mesh filename=./assets/wujihand_full/left/left_finger2_link3.STL
- link left_finger2_link4: geometry collision mesh filename=./assets/wujihand_full_simplified_v1/left/left_finger2_link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; visual mesh filename=./assets/wujihand_full/left/left_finger2_link4.STL
- link left_finger3_link1: geometry collision mesh filename=./assets/wujihand_full_simplified_v1/left/left_finger3_link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; collision mesh filename=./assets/wujihand_full_simplified_v1/left/left_finger3_link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
- link left_finger3_link2: geometry collision mesh filename=./assets/wujihand_full_simplified_v1/left/left_finger3_link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; visual mesh filename=./assets/wujihand_full/left/left_finger3_link2.STL
- link left_finger3_link3: geometry collision mesh filename=./assets/wujihand_full_simplified_v1/left/left_finger3_link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; visual mesh filename=./assets/wujihand_full/left/left_finger3_link3.STL
- link left_finger3_link4: geometry collision mesh filename=./assets/wujihand_full_simplified_v1/left/left_finger3_link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; visual mesh filename=./assets/wujihand_full/left/left_finger3_link4.STL
- link left_finger4_link1: geometry collision mesh filename=./assets/wujihand_full_simplified_v1/left/left_finger4_link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; collision mesh filename=./assets/wujihand_full_simplified_v1/left/left_finger4_link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
- link left_finger4_link2: geometry collision mesh filename=./assets/wujihand_full_simplified_v1/left/left_finger4_link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; visual mesh filename=./assets/wujihand_full/left/left_finger4_link2.STL
- link left_finger4_link3: geometry collision mesh filename=./assets/wujihand_full_simplified_v1/left/left_finger4_link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; visual mesh filename=./assets/wujihand_full/left/left_finger4_link3.STL
- link left_finger4_link4: geometry collision mesh filename=./assets/wujihand_full_simplified_v1/left/left_finger4_link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; visual mesh filename=./assets/wujihand_full/left/left_finger4_link4.STL
- link left_finger5_link1: geometry collision mesh filename=./assets/wujihand_full_simplified_v1/left/left_finger5_link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; collision mesh filename=./assets/wujihand_full_simplified_v1/left/left_finger5_link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
- link left_finger5_link2: geometry collision mesh filename=./assets/wujihand_full_simplified_v1/left/left_finger5_link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; visual mesh filename=./assets/wujihand_full/left/left_finger5_link2.STL
- link left_finger5_link3: geometry collision mesh filename=./assets/wujihand_full_simplified_v1/left/left_finger5_link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; visual mesh filename=./assets/wujihand_full/left/left_finger5_link3.STL
- link left_finger5_link4: geometry collision mesh filename=./assets/wujihand_full_simplified_v1/left/left_finger5_link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; collision mesh filename=./assets/wujihand_full_simplified_v1/left/left_finger5_link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
- link left_palm_link: geometry collision mesh filename=./assets/wujihand_full_simplified_v1/left/left_palm_link/le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; visual mesh filename=./assets/wujihand_full/left/left_palm_link.STL

File: source/regrind/regrind/assets/mjcf/free_wuji_left_hand_full_simplified_v1_render.urdf (robot description, URDF)
Before this commit: robot wujihand-left, 48 links, 47 joints
Links:
- link left_finger1_link1: geometry collision mesh filename=./assets/wujihand_full_simplified_v1/left/left_finger1_link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; collision mesh filename=./assets/wujihand_full_simplified_v1/left/left_finger1_link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
- link left_finger1_link2: geometry collision mesh filename=./assets/wujihand_full_simplified_v1/left/left_finger1_link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; visual mesh filename=./assets/wujihand_full/left/left_finger1_link2.obj
- link left_finger1_link3: geometry collision mesh filename=./assets/wujihand_full_simplified_v1/left/left_finger1_link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; visual mesh filename=./assets/wujihand_full/left/left_finger1_link3.obj
- link left_finger1_link4: geometry collision mesh filename=./assets/wujihand_full_simplified_v1/left/left_finger1_link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; visual mesh filename=./assets/wujihand_full/left/left_finger1_link4.obj
- link left_finger2_link1: geometry collision mesh filename=./assets/wujihand_full_simplified_v1/left/left_finger2_link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; collision mesh filename=./assets/wujihand_full_simplified_v1/left/left_finger2_link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
- link left_finger2_link2: geometry collision mesh filename=./assets/wujihand_full_simplified_v1/left/left_finger2_link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; visual mesh filename=./assets/wujihand_full/left/left_finger2_link2.obj
- link left_finger2_link3: geometry collision mesh filename=./assets/wujihand_full_simplified_v1/left/left_finger2_link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; visual mesh filename=./assets/wujihand_full/left/left_finger2_link3.obj
- link left_finger2_link4: geometry collision mesh filename=./assets/wujihand_full_simplified_v1/left/left_finger2_link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; visual mesh filename=./assets/wujihand_full/left/left_finger2_link4.obj
- link left_finger3_link1: geometry collision mesh filename=./assets/wujihand_full_simplified_v1/left/left_finger3_link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; collision mesh filename=./assets/wujihand_full_simplified_v1/left/left_finger3_link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
- link left_finger3_link2: geometry collision mesh filename=./assets/wujihand_full_simplified_v1/left/left_finger3_link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; visual mesh filename=./assets/wujihand_full/left/left_finger3_link2.obj
- link left_finger3_link3: geometry collision mesh filename=./assets/wujihand_full_simplified_v1/left/left_finger3_link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; visual mesh filename=./assets/wujihand_full/left/left_finger3_link3.obj
- link left_finger3_link4: geometry collision mesh filename=./assets/wujihand_full_simplified_v1/left/left_finger3_link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; visual mesh filename=./assets/wujihand_full/left/left_finger3_link4.obj
- link left_finger4_link1: geometry collision mesh filename=./assets/wujihand_full_simplified_v1/left/left_finger4_link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; collision mesh filename=./assets/wujihand_full_simplified_v1/left/left_finger4_link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
- link left_finger4_link2: geometry collision mesh filename=./assets/wujihand_full_simplified_v1/left/left_finger4_link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; visual mesh filename=./assets/wujihand_full/left/left_finger4_link2.obj
- link left_finger4_link3: geometry collision mesh filename=./assets/wujihand_full_simplified_v1/left/left_finger4_link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; visual mesh filename=./assets/wujihand_full/left/left_finger4_link3.obj
- link left_finger4_link4: geometry collision mesh filename=./assets/wujihand_full_simplified_v1/left/left_finger4_link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; visual mesh filename=./assets/wujihand_full/left/left_finger4_link4.obj
- link left_finger5_link1: geometry collision mesh filename=./assets/wujihand_full_simplified_v1/left/left_finger5_link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; collision mesh filename=./assets/wujihand_full_simplified_v1/left/left_finger5_link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
- link left_finger5_link2: geometry collision mesh filename=./assets/wujihand_full_simplified_v1/left/left_finger5_link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; visual mesh filename=./assets/wujihand_full/left/left_finger5_link2.obj
- link left_finger5_link3: geometry collision mesh filename=./assets/wujihand_full_simplified_v1/left/left_finger5_link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; visual mesh filename=./assets/wujihand_full/left/left_finger5_link3.obj
- link left_finger5_link4: geometry collision mesh filename=./assets/wujihand_full_simplified_v1/left/left_finger5_link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; collision mesh filename=./assets/wujihand_full_simplified_v1/left/left_finger5_link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
- link left_palm_link: geometry collision mesh filename=./assets/wujihand_full_simplified_v1/left/left_palm_link/le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; visual mesh filename=./assets/wujihand_full/left/left_palm_link.obj
