Commit message: Wrist-calibrate left base_joint, corrected formula (verified)
Correct transform: R(G')=Cr*Cl^-1*R(G), t(G')=Cr^-1(dl-dr)+R(G')R(G)^-1 t(G),
computed from ORIGINAL models' measured offsets. Previous commit used the wrong
composition order (oscillated 160->40->82deg). Verified on 200-frame runs:
wujihand_left 159.6->8.9deg (right ref 5.4), leaphand_left 111->32.4deg
(right ref 26.3); joint err unchanged ~2-3cm.

File: source/regrind/regrind/assets/leaphand_urdf/leap_hand_left_mano.urdf (robot description, URDF)
Before this commit: robot leap_left, 35 links, 34 joints
Joints:
- joint base_joint: origin xyz=-0.130455 -0.105818 0.054945 rpy=2.691491 0.071008 -2.105230 -> xyz=0.111523 0.139473 -0.035494 rpy=-1.499563 0.054832 0.858888

File: source/regrind/regrind/assets/leaphand_urdf/leap_hand_left_render.urdf (robot description, URDF)
Before this commit: robot leap_left, 35 links, 34 joints
Joints:
- joint base_joint: origin xyz=-0.130455 -0.105818 0.054945 rpy=2.691491 0.071008 -2.105230 -> xyz=0.111523 0.139473 -0.035494 rpy=-1.499563 0.054832 0.858888

File: source/regrind/regrind/assets/mjcf/free_wuji_left_hand_full_simplified_v1.urdf (robot description, URDF)
Before this commit: robot wujihand-left, 48 links, 47 joints
Joints:
- joint base_joint: origin xyz=-0.006209 0.012544 0.046687 rpy=-2.745849 1.252560 2.359086 -> xyz=0.004128 0.014200 0.044564 rpy=-2.699035 1.409043 1.624471

File: source/regrind/regrind/assets/mjcf/free_wuji_left_hand_full_simplified_v1_render.urdf (robot description, URDF)
Before this commit: robot wujihand-left, 48 links, 47 joints
Joints:
- joint base_joint: origin xyz=-0.006209 0.012544 0.046687 rpy=-2.745849 1.252560 2.359086 -> xyz=0.004128 0.014200 0.044564 rpy=-2.699035 1.409043 1.624471

Commit message: leaphand_left base_joint v4 (T_r^-1 T_off G, 2 iters) + left render meshes
- v4 calibration vs clean right baseline (drink_bowl_R 24.8deg/11mm):
  smoke cut_knife_L 34deg -> 27.4+/-6.3deg, translation 35.7 -> 10.5mm;
  leap anchors verified NOT broken (L/R-consistent ~8mm, correct chirality)
- add meshes/visual_normals for the left render URDF (normals-carrying OBJs,
  Blender black_metal mtl stripped -> uniform Drake default shading)

File: source/regrind/regrind/assets/leaphand_urdf/leap_hand_left_mano.urdf (robot description, URDF)
Before this commit: robot leap_left, 35 links, 34 joints
Joints:
- joint base_joint: origin xyz=0.111523 0.139473 -0.035494 rpy=-1.499563 0.054832 0.858888 -> xyz=0.117340 0.105773 -0.049289 rpy=-1.338486 0.099190 0.759435

File: source/regrind/regrind/assets/leaphand_urdf/leap_hand_left_render.urdf (robot description, URDF)
Before this commit: robot leap_left, 35 links, 34 joints
Joints:
- joint base_joint: origin xyz=0.111523 0.139473 -0.035494 rpy=-1.499563 0.054832 0.858888 -> xyz=0.117340 0.105773 -0.049289 rpy=-1.338486 0.099190 0.759435
