Commit message: assets: rename knife visual mesh (USD SdfPath rejects digit-leading '3DModel')

File: source/regrind/regrind/assets/tactidex/knife/knife.urdf (robot description, URDF)
Before this commit: robot knife, 1 links, 0 joints
Links:
- link bottom: geometry collision mesh filename=collision_parts/part_000.obj scale=1 1 1; collision mesh filename=collision_parts/part_001.obj scale=1 1 1
